Commit message: Spremenjem node marker.cpp za povezovanje podatkov /scan in camera trenutno poda poda razdaljo od zaznage objekta

File: simulation/models/urdf/robot1.xacro (robot description, xacro)
@@ -64,5 +64,5 @@
     </link>
     <joint name="camera_joint" type="fixed">
-        <origin xyz="0.3 0.2 0.2" rpy="0 0 0"/>
+        <origin xyz="0.3 0 0.25" rpy="0 0 0"/>
         <parent link="base_link"/>
         <child link="camera_link"/>

Commit message: Dodant node za kalibracijo kamere in lidarja

File: simulation/models/urdf/robot1.xacro (robot description, xacro)
@@ -64,5 +64,5 @@
     </link>
     <joint name="camera_joint" type="fixed">
-        <origin xyz="0.3 0 0.25" rpy="0 0 0"/>
+        <origin xyz="0.3 0.15 0.25" rpy="0 0 0"/>
         <parent link="base_link"/>
         <child link="camera_link"/>
